File: board/src/chrimbus/chrimbus.sch (KiCad schematic (older format))
At the start: 37 parts, among them J1 Conn_01x06, SW1 SW_SPST, U1 PIC16F15325, U2 XC9142, U3 TLC59116F

Commit message: last commit before dev branch
Parts:
- added C4: 0.1uF, Capacitor_SMD:C_0805_2012Metric, symbol Device:C
- added MH1: MountingHole, MountingHole:MountingHole_2.2mm_M2, symbol Mechanical:MountingHole
Connections:
- net +3V3: now also C4.2
- net GND: now also C4.1
Changed lines of the file:
@@
 EESchema Schematic File Version 4
+LIBS:chrimbus-cache
 EELAYER 26 0
 EELAYER END
@@
 	6750 2400 6750 2550
 Wire Wire Line
-	6400 2850 6750 2850
+	6400 2850 6550 2850
 $Comp
 L Device:R R21
@@
 Wire Wire Line
 	6100 3700 6100 3850
+$Comp
+L Device:C C4
+U 1 1 5BFA64D0
+P 6550 2700
+F 0 "C4" V 6298 2700 50  0000 C CNN
+F 1 "0.1uF" V 6389 2700 50  0000 C CNN
+F 2 "Capacitor_SMD:C_0805_2012Metric" H 6588 2550 50  0001 C CNN
+F 3 "~" H 6550 2700 50  0001 C CNN
+	1    6550 2700
+	-1   0    0    1
+$EndComp
+Connection ~ 6550 2850
+Wire Wire Line
+	6550 2850 6750 2850
+Wire Wire Line
+	6550 2550 6750 2550
+Connection ~ 6750 2550
+$Comp
+L Mechanical:MountingHole MH1
+U 1 1 5BFB160D
+P 5400 1900
+F 0 "MH1" H 5500 1946 50  0000 L CNN
+F 1 "MountingHole" H 5500 1855 50  0000 L CNN
+F 2 "MountingHole:MountingHole_2.2mm_M2" H 5400 1900 50  0001 C CNN
+F 3 "~" H 5400 1900 50  0001 C CNN
+	1    5400 1900
+	1    0    0    -1
+$EndComp
 $EndSCHEMATC
