File: board/src/chrimbus/chrimbus.kicad_pcb (KiCad board)
At the start: 2 copper layers, 90 x 89.7 mm, 37 parts, among them J1 Conn_01x06, SW1 SW_SPST, U1 PIC16F15325, U2 XC9142, U3 TLC59116F

Commit message: last commit before dev branch
Parts:
- added C4: 0.1uF, Capacitor_SMD:C_0805_2012Metric, F.Cu at (163.9, 100.3)
- added MH1: MountingHole, MountingHole:MountingHole_2.2mm_M2, F.Cu at (167.1, 57.4)
- moved R20 5.60 mm to (166.6, 62.6), turned to 0 degrees
- moved LED6 2.05 mm to (164.9, 61.0)
Routing:
- net +1V5: track 0.00 -> 51.3 mm
- net Net-(C1-Pad2): track 7.54 -> 42.5 mm, vias 0 -> 1
- net GND: track 7.41 -> 41.0 mm, vias 0 -> 6
- net Net-(R17-Pad2): track 0.00 -> 33.0 mm, vias 0 -> 2
- net Net-(R18-Pad2): track 0.00 -> 29.7 mm, vias 0 -> 2
- net Net-(R19-Pad2): track 0.00 -> 26.8 mm, vias 0 -> 2
- net +3V3: track 0.00 -> 23.3 mm, vias 0 -> 3
- net Net-(R20-Pad2): track 43.3 -> 50.5 mm
- net Net-(LED6-Pad1): track 4.06 -> 2.04 mm
- added copper zone on B.Cu, net GND
Other:
- board text added: "*"
- board text added: "2018"
- board text added: "LOVE, JAKE"
- board text added: "MERRY CHRISTMAS!"
- board text removed: "MERRY CHRISTMAS 2018 <3 JAKE"

Commit message: dev final commit
Parts:
- moved L1 5.50 mm to (170.0, 88.4), turned to 90 degrees
- moved R2 2.18 mm to (167.0, 91.6)
- moved C3 0.48 mm to (162.5, 88.4), turned to 270 degrees
Connections:
- U2 pad 1: Net-(R2-Pad2) -> Net-(L1-Pad1)
- U2 pad 2: GND -> Net-(R2-Pad2)
- U2 pad 4: +3V3 -> GND
- U2 pad 5: Net-(L1-Pad1) -> +3V3
Routing:
- net GND: track 41.0 -> 44.4 mm, vias 6 -> 5
- net Net-(R16-Pad2): track 26.7 -> 29.1 mm
- net +3V3: track 23.3 -> 25.5 mm
- net Net-(R2-Pad2): track 2.98 -> 4.37 mm
- net Net-(C1-Pad2): track 42.5 -> 43.2 mm
